File: kicad_buck_converter/buck_converter.kicad_sch (KiCad schematic)
At the start: 8 parts, among them J1 Input, J2 Output, U1 LM2596S-5.0

Commit message: update branch
Parts:
- removed U?: (no value)
Changed lines of the file:
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@@
 (kicad_sch (version 20240108) (generator kicad_sch_symbol_editor)
-  (symbol (lib_id "") (at 0 0)
-    (in_bom yes) (on_board yes)
-    (property "Reference" "U?" (at 0 0) (effects (font (size 1.27 1.27))))
-  )
-  (sheet (at 0 0) (size 297 210) (stroke (width 0) (type default)) (fill (type none))
+  (sheet (at 0 0) (size 297 210) (stroke (width 0.15)) (fill (type background))
     (property "Reference" "" (at 0 0) (effects (font (size 1.27 1.27))))
   )
@@
     (date "2025-01-13")
   )
-  (symbol (lib_id "Device:C_Polarized_US") (at 50 50) (unit 1)
+  (symbol (lib_id "Device:C_Polarized_US") (at 50 50 0) (unit 1)
     (in_bom yes) (on_board yes)
     (property "Reference" "C1" (at 50 65) (effects (font (size 1.27 1.27))))
@@
     (property "Footprint" "Capacitor_THT:CP_Radial_D5.0mm_P2.50mm" (at 50 85) (effects (font (size 1.27 1.27)) hide))
   )
-  (symbol (lib_id "Device:C_Polarized_US") (at 150 100) (unit 1)
+  (symbol (lib_id "Device:C_Polarized_US") (at 150 100 0) (unit 1)
     (in_bom yes) (on_board yes)
     (property "Reference" "C2" (at 150 115) (effects (font (size 1.27 1.27))))
@@
     (property "Footprint" "Capacitor_THT:CP_Radial_D5.0mm_P2.50mm" (at 150 135) (effects (font (size 1.27 1.27)) hide))
   )
-  (symbol (lib_id "Device:L_Core_Ferrite_US") (at 100 50) (unit 1)
+  (symbol (lib_id "Device:L_Core_Ferrite_US") (at 100 50 0) (unit 1)
     (in_bom yes) (on_board yes)
     (property "Reference" "L1" (at 100 35) (effects (font (size 1.27 1.27))))
@@
     (property "Footprint" "Inductor_THT:L_Radial_D5.0mm_P2.50mm" (at 100 15) (effects (font (size 1.27 1.27)) hide))
   )
-  (symbol (lib_id "Diode:D_Schottky_US") (at 100 100) (unit 1)
+  (symbol (lib_id "Diode:D_Schottky_US") (at 100 100 0) (unit 1)
     (in_bom yes) (on_board yes)
     (property "Reference" "D1" (at 100 85) (effects (font (size 1.27 1.27))))
@@
     (property "Footprint" "Diode_THT:D_DO-214AC_SMA_Horizontal" (at 100 65) (effects (font (size 1.27 1.27)) hide))
   )
-  (symbol (lib_id "Regulator_Switching:LM2596S-5.0") (at 75 75) (unit 1)
+  (symbol (lib_id "Regulator_Switching:LM2596S-5.0") (at 75 75 0) (unit 1)
     (in_bom yes) (on_board yes)
     (property "Reference" "U1" (at 75 60) (effects (font (size 1.27 1.27))))
@@
     (property "Footprint" "Package_TO_SOT_SMD:TO-263-5" (at 75 40) (effects (font (size 1.27 1.27)) hide))
   )
-  (symbol (lib_id "Connector:Conn_01x02_Male") (at 20 50) (unit 1)
+  (symbol (lib_id "Connector:Conn_01x02_Male") (at 20 50 0) (unit 1)
     (in_bom yes) (on_board yes)
     (property "Reference" "J1" (at 20 35) (effects (font (size 1.27 1.27))))
@@
     (property "Footprint" "TerminalBlock_Phoenix:TerminalBlock_Phoenix_MKDSN-2-5.08_2x5.08mm_Angled" (at 20 15) (effects (font (size 1.27 1.27)) hide))
   )
-  (symbol (lib_id "Connector:Conn_01x02_Male") (at 200 100) (unit 1)
+  (symbol (lib_id "Connector:Conn_01x02_Male") (at 200 100 0) (unit 1)
     (in_bom yes) (on_board yes)
     (property "Reference" "J2" (at 200 85) (effects (font (size 1.27 1.27))))

Commit message: update branch
Other:
- removed sheet 
- note removed: "GND"
- note removed: "VIN"
- note removed: "VOUT"
Changed lines of the file:
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@@
 (kicad_sch (version 20240108) (generator kicad_sch_symbol_editor)
-  (sheet (at 0 0) (size 297 210) (stroke (width 0.15)) (fill (type background))
-    (property "Reference" "" (at 0 0) (effects (font (size 1.27 1.27))))
-  )
+  (paper "A4")
   (title_block
     (title "Buck Converter LM2596")
@@
   (symbol (lib_id "Device:C_Polarized_US") (at 50 50 0) (unit 1)
     (in_bom yes) (on_board yes)
-    (property "Reference" "C1" (at 50 65) (effects (font (size 1.27 1.27))))
-    (property "Value" "10uF" (at 50 75) (effects (font (size 1.27 1.27))))
-    (property "Footprint" "Capacitor_THT:CP_Radial_D5.0mm_P2.50mm" (at 50 85) (effects (font (size 1.27 1.27)) hide))
+    (property "Reference" "C1" (at 50 65 0) (effects (font (size 1.27 1.27))))
+    (property "Value" "10uF" (at 50 75 0) (effects (font (size 1.27 1.27))))
+    (property "Footprint" "Capacitor_THT:CP_Radial_D5.0mm_P2.50mm" (at 50 85 0) (effects (font (size 1.27 1.27)) hide))
   )
   (symbol (lib_id "Device:C_Polarized_US") (at 150 100 0) (unit 1)
     (in_bom yes) (on_board yes)
-    (property "Reference" "C2" (at 150 115) (effects (font (size 1.27 1.27))))
-    (property "Value" "22uF" (at 150 125) (effects (font (size 1.27 1.27))))
-    (property "Footprint" "Capacitor_THT:CP_Radial_D5.0mm_P2.50mm" (at 150 135) (effects (font (size 1.27 1.27)) hide))
+    (property "Reference" "C2" (at 150 115 0) (effects (font (size 1.27 1.27))))
+    (property "Value" "22uF" (at 150 125 0) (effects (font (size 1.27 1.27))))
+    (property "Footprint" "Capacitor_THT:CP_Radial_D5.0mm_P2.50mm" (at 150 135 0) (effects (font (size 1.27 1.27)) hide))
   )
   (symbol (lib_id "Device:L_Core_Ferrite_US") (at 100 50 0) (unit 1)
     (in_bom yes) (on_board yes)
-    (property "Reference" "L1" (at 100 35) (effects (font (size 1.27 1.27))))
-    (property "Value" "10uH" (at 100 25) (effects (font (size 1.27 1.27))))
-    (property "Footprint" "Inductor_THT:L_Radial_D5.0mm_P2.50mm" (at 100 15) (effects (font (size 1.27 1.27)) hide))
+    (property "Reference" "L1" (at 100 35 0) (effects (font (size 1.27 1.27))))
+    (property "Value" "10uH" (at 100 25 0) (effects (font (size 1.27 1.27))))
+    (property "Footprint" "Inductor_THT:L_Radial_D5.0mm_P2.50mm" (at 100 15 0) (effects (font (size 1.27 1.27)) hide))
   )
   (symbol (lib_id "Diode:D_Schottky_US") (at 100 100 0) (unit 1)
     (in_bom yes) (on_board yes)
-    (property "Reference" "D1" (at 100 85) (effects (font (size 1.27 1.27))))
-    (property "Value" "SS34" (at 100 75) (effects (font (size 1.27 1.27))))
-    (property "Footprint" "Diode_THT:D_DO-214AC_SMA_Horizontal" (at 100 65) (effects (font (size 1.27 1.27)) hide))
+    (property "Reference" "D1" (at 100 85 0) (effects (font (size 1.27 1.27))))
+    (property "Value" "SS34" (at 100 75 0) (effects (font (size 1.27 1.27))))
+    (property "Footprint" "Diode_THT:D_DO-214AC_SMA_Horizontal" (at 100 65 0) (effects (font (size 1.27 1.27)) hide))
   )
   (symbol (lib_id "Regulator_Switching:LM2596S-5.0") (at 75 75 0) (unit 1)
     (in_bom yes) (on_board yes)
-    (property "Reference" "U1" (at 75 60) (effects (font (size 1.27 1.27))))
-    (property "Value" "LM2596S-5.0" (at 75 50) (effects (font (size 1.27 1.27))))
-    (property "Footprint" "Package_TO_SOT_SMD:TO-263-5" (at 75 40) (effects (font (size 1.27 1.27)) hide))
+    (property "Reference" "U1" (at 75 60 0) (effects (font (size 1.27 1.27))))
+    (property "Value" "LM2596S-5.0" (at 75 50 0) (effects (font (size 1.27 1.27))))
+    (property "Footprint" "Package_TO_SOT_SMD:TO-263-5" (at 75 40 0) (effects (font (size 1.27 1.27)) hide))
   )
   (symbol (lib_id "Connector:Conn_01x02_Male") (at 20 50 0) (unit 1)
     (in_bom yes) (on_board yes)
-    (property "Reference" "J1" (at 20 35) (effects (font (size 1.27 1.27))))
-    (property "Value" "Input" (at 20 25) (effects (font (size 1.27 1.27))))
-    (property "Footprint" "TerminalBlock_Phoenix:TerminalBlock_Phoenix_MKDSN-2-5.08_2x5.08mm_Angled" (at 20 15) (effects (font (size 1.27 1.27)) hide))
+    (property "Reference" "J1" (at 20 35 0) (effects (font (size 1.27 1.27))))
+    (property "Value" "Input" (at 20 25 0) (effects (font (size 1.27 1.27))))
+    (property "Footprint" "TerminalBlock_Phoenix:TerminalBlock_Phoenix_MKDSN-2-5.08_2x5.08mm_Angled" (at 20 15 0) (effects (font (size 1.27 1.27)) hide))
   )
   (symbol (lib_id "Connector:Conn_01x02_Male") (at 200 100 0) (unit 1)
     (in_bom yes) (on_board yes)
-    (property "Reference" "J2" (at 200 85) (effects (font (size 1.27 1.27))))
-    (property "Value" "Output" (at 200 75) (effects (font (size 1.27 1.27))))
-    (property "Footprint" "TerminalBlock_Phoenix:TerminalBlock_Phoenix_MKDSN-2-5.08_2x5.08mm_Angled" (at 200 65) (effects (font (size 1.27 1.27)) hide))
+    (property "Reference" "J2" (at 200 85 0) (effects (font (size 1.27 1.27))))
+    (property "Value" "Output" (at 200 75 0) (effects (font (size 1.27 1.27))))
+    (property "Footprint" "TerminalBlock_Phoenix:TerminalBlock_Phoenix_MKDSN-2-5.08_2x5.08mm_Angled" (at 200 65 0) (effects (font (size 1.27 1.27)) hide))
   )
-  (junction (at 75 50) (diameter 0) (color 0 0 0 0)
-  )
-  (junction (at 100 50) (diameter 0) (color 0 0 0 0)
-  )
-  (junction (at 150 100) (diameter 0) (color 0 0 0 0)
-  )
-  (wire (pts (xy 30 50) (xy 50 50))
-    (stroke (width 0) (type default))
-  )
-  (wire (pts (xy 50 50) (xy 75 50))
-    (stroke (width 0) (type default))
-  )
-  (wire (pts (xy 75 50) (xy 100 50))
-    (stroke (width 0) (type default))
-  )
-  (wire (pts (xy 100 50) (xy 120 50))
-    (stroke (width 0) (type default))
-  )
-  (wire (pts (xy 150 100) (xy 180 100))
-    (stroke (width 0) (type default))
-  )
-  (wire (pts (xy 100 100) (xy 150 100))
-    (stroke (width 0) (type default))
-  )
-  (no_connect (at 120 50)
-  )
-  (text "VIN" (at 25 45) (effects (font (size 1.27 1.27)))
-  )
-  (text "VOUT" (at 185 95) (effects (font (size 1.27 1.27)))
-  )
-  (text "GND" (at 50 80) (effects (font (size 1.27 1.27)))
-  )
-  (text "GND" (at 150 130) (effects (font (size 1.27 1.27)))
-  )
+  (junction (at 75 50) (diameter 0) (color 0 0 0 0))
+  (junction (at 100 50) (diameter 0) (color 0 0 0 0))
+  (junction (at 150 100) (diameter 0) (color 0 0 0 0))
+  (wire (pts (xy 30 50) (xy 50 50)) (stroke (width 0) (type default)))
+  (wire (pts (xy 50 50) (xy 75 50)) (stroke (width 0) (type default)))
+  (wire (pts (xy 75 50) (xy 100 50)) (stroke (width 0) (type default)))
+  (wire (pts (xy 100 50) (xy 120 50)) (stroke (width 0) (type default)))
+  (wire (pts (xy 150 100) (xy 180 100)) (stroke (width 0) (type default)))
+  (wire (pts (xy 100 100) (xy 150 100)) (stroke (width 0) (type default)))
+  (no_connect (at 120 50))
+  (label "VIN" (at 25 45 0) (effects (font (size 1.27 1.27))))
+  (label "VOUT" (at 185 95 0) (effects (font (size 1.27 1.27))))
+  (label "GND" (at 50 80 0) (effects (font (size 1.27 1.27))))
+  (label "GND" (at 150 130 0) (effects (font (size 1.27 1.27))))
 )
